Commit message: add controller launch.

File: src/arduinobot_description/urdf/arduinobot.urdf.xacro (robot description, xacro)
@@ -142,5 +142,5 @@
         <origin xyz="0 0 0" rpy="0 0 0"/>
     </joint>
-    <joint name ="joint_1" type="revolute">
+    <joint name="joint_1" type="revolute">
         <parent link="base_link"/>
         <child link = "base_plate"/>
@@ -149,5 +149,5 @@
         <limit lower="-${PI/2}" upper="${PI/2}" effort="${effort}" velocity="${velocity}"/>
     </joint>
-    <joint name ="joint_2" type="revolute">
+    <joint name="joint_2" type="revolute">
         <parent link="base_plate"/>
         <child link = "forward_drive_arm"/>
@@ -156,5 +156,5 @@
         <limit lower="-${PI/2}" upper="${PI/2}" effort="${effort}" velocity="${velocity}"/>
     </joint>
-    <joint name ="joint_3" type="revolute">
+    <joint name="joint_3" type="revolute">
         <parent link="forward_drive_arm"/>
         <child link = "horizontal_arm"/>
@@ -163,10 +163,10 @@
         <limit lower="-${PI/2}" upper="${PI/2}" effort="${effort}" velocity="${velocity}"/>
     </joint>
-    <joint name ="horizontal_arm_to_claw_support" type="fixed">
+    <joint name="horizontal_arm_to_claw_support" type="fixed">
         <parent link="horizontal_arm"/>
         <child link = "claw_support"/>
         <origin xyz="0 0.82 0"/>
     </joint>
-    <joint name ="joint_4" type="revolute">
+    <joint name="joint_4" type="revolute">
         <parent link="claw_support"/>
         <child link = "gripper_right"/>
@@ -175,5 +175,5 @@
         <limit lower="-${PI/2}" upper="0" effort="${effort}" velocity="${velocity}"/>
     </joint>
-    <joint name ="joint_5" type="revolute">
+    <joint name="joint_5" type="revolute">
         <parent link="claw_support"/>
         <child link = "gripper_left"/>
