Commit message: add the pen to the scene

File: arduinobot.urdf (robot description, URDF)
Before this commit: robot arduinobot, 9 links, 8 joints
Links:
- link base_link: mass None -> 1; geometry collision mesh filename=package://arduinobot_description/mesh/basement.STL scale=0.01 0.01 0.01; visual mesh filename=package://arduinobot_description/mesh/basement.STL scale=0.01 0.01 0.01
- link base_plate: mass None -> 0.1; geometry collision mesh filename=package://arduinobot_description/mesh/base_plate.STL scale=0.01 0.01 0.01; visual mesh filename=package://arduinobot_description/mesh/base_plate.STL scale=0.01 0.01 0.01
- link claw_support: mass None -> 0.05; geometry collision mesh filename=package://arduinobot_description/mesh/claw_support.STL scale=0.01 0.01 0.01; visual mesh filename=package://arduinobot_description/mesh/claw_support.STL scale=0.01 0.01 0.01
- link forward_drive_arm: mass None -> 0.1; geometry collision mesh filename=package://arduinobot_description/mesh/forward_drive_arm.STL scale=0.01 0.01 0.01; visual mesh filename=package://arduinobot_description/mesh/forward_drive_arm.STL scale=0.01 0.01 0.01
- link gripper_left: mass None -> 0.01; geometry collision mesh filename=package://arduinobot_description/mesh/left_finger.STL scale=0.01 0.01 0.01; visual mesh filename=package://arduinobot_description/mesh/left_finger.STL scale=0.01 0.01 0.01
- link gripper_right: mass None -> 0.01; geometry collision mesh filename=package://arduinobot_description/mesh/right_finger.STL scale=0.01 0.01 0.01; visual mesh filename=package://arduinobot_description/mesh/right_finger.STL scale=0.01 0.01 0.01
- link horizontal_arm: mass None -> 0.1; geometry collision mesh filename=package://arduinobot_description/mesh/horizontal_arm.STL scale=0.01 0.01 0.01; visual mesh filename=package://arduinobot_description/mesh/horizontal_arm.STL scale=0.01 0.01 0.01

File: src/arduinobot_description/urdf/arduinobot.urdf.xacro (robot description, xacro)
@@ -135,5 +135,21 @@
         </collision>
     </link>
-    <link name="tool_link"></link>
+    <link name="tool_link">
+        <link name="tool_link">
+            <xacro:default_inertial mass="0.01"/>
+            <visual>
+                <origin rpy="0 0 -${PI/2}" xyz="-0.04 0.50 -0.1"/>
+                <geometry>
+                    <cylinder radius="0.03" length="1.0"/>
+                </geometry>
+            </visual>
+            <collision>
+                <origin rpy="0 0 -${PI/2}" xyz="-0.04 0.50 -0.1"/>
+                <geometry>
+                    <cylinder radius="0.03" length="1.0"/>
+                </geometry>
+            </collision>
+        </link>
+    </link>
     <!-- Joints -->
     <joint name="virtual_joint" type="fixed">
